File: pcb/test-signal-interface.kicad_sch (KiCad schematic)
At the start: 7 parts, among them J4 BSE-040-01-F-D-A-TR, J5 BSE-040-01-F-D-A-TR, U1 AT24C64D-SSHM-T

Commit message: Revision B
- Added 220k resistor arrays in series with amplifier connections to
  simulate electrodes
Changed lines of the file:
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@@
 	(title_block
 		(title "Ephys Test Module - 64 Channel (MOLC)")
-		(rev "A")
+		(rev "B")
 		(company "Open Ephys, Inc.")
 	)
@@
 					(size 1.27 1.27)
 				)
-				(hide yes)
 			)
 		)
@@
 					(size 1.27 1.27)
 				)
-				(hide yes)
 			)
 		)
@@
 					(size 1.27 1.27)
 				)
-				(hide yes)
 			)
 		)

Commit message: Revision B
- Widened traces to 0.2 mm
Parts:
- C1: TempCo X7R -> (none); Tolerance (none) -> X5R
- R1, R2, R3: Tolerance (none) -> 1%
Changed lines of the file:
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@@
+			)
+		)
+		(property "Temp. Co." ""
+			(at 91.44 76.2 0)
+			(effects
+				(font
+					(size 1.27 1.27)
+				)
+				(hide yes)
 			)
 		)
@@
 			)
 		)
+		(property "Temp. Co." ""
+			(at 196.85 76.2 0)
+			(effects
+				(font
+					(size 1.27 1.27)
+				)
+				(hide yes)
+			)
+		)
 		(pin "1"
 		)
@@
 			)
 		)
-		(property "Tolerance" ""
+		(property "Tolerance" "1%"
 			(at 60.96 162.56 0)
 			(effects
@@
 		)
 		(property "OEPSPN" "OEPS020027"
+			(at 60.96 162.56 0)
+			(effects
+				(font
+					(size 1.27 1.27)
+				)
+				(hide yes)
+			)
+		)
+		(property "Temp. Co." ""
 			(at 60.96 162.56 0)
 			(effects
@@
 			)
 		)
-		(property "Tolerance" ""
+		(property "Tolerance" "1%"
 			(at 69.85 162.56 0)
 			(effects
@@
 		)
 		(property "OEPSPN" "OEPS020027"
+			(at 69.85 162.56 0)
+			(effects
+				(font
+					(size 1.27 1.27)
+				)
+				(hide yes)
+			)
+		)
+		(property "Temp. Co." ""
 			(at 69.85 162.56 0)
 			(effects
@@
 			)
 		)
-		(property "Tolerance" ""
+		(property "Tolerance" "1%"
 			(at 78.74 162.56 0)
 			(effects
@@
 		)
 		(property "OEPSPN" "OEPS020027"
+			(at 78.74 162.56 0)
+			(effects
+				(font
+					(size 1.27 1.27)
+				)
+				(hide yes)
+			)
+		)
+		(property "Temp. Co." ""
 			(at 78.74 162.56 0)
 			(effects
@@
 			)
 		)
+		(property "Temp. Co." ""
+			(at 107.95 172.72 0)
+			(effects
+				(font
+					(size 1.27 1.27)
+				)
+				(hide yes)
+			)
+		)
 		(pin "1"
 		)
@@
 			)
 		)
-		(property "TempCo" "X7R"
-			(at 115.57 162.56 0)
-			(effects
-				(font
-					(size 1.27 1.27)
-				)
-				(hide yes)
-			)
-		)
 		(property "Voltage" ""
 			(at 115.57 162.56 0)
@@
 			)
 		)
-		(property "Tolerance" ""
+		(property "Tolerance" "X5R"
 			(at 115.57 162.56 0)
 			(effects
@@
 			(effects
 				(font
+					(size 1.27 1.27)
+				)
+				(hide yes)
+			)
+		)
+		(property "Temp. Co." ""
+			(at 115.57 162.56 90)
+			(effects
+				(font
